File: esp32pcbbot.kicad_pcb (KiCad board)
At the start: 2 copper layers, 110 x 170 mm, 44 parts, among them IC1 BMI055, J1 TB002-500-02BE, J2 TB002-500-02BE, J3 TB002-500-02BE, J4 215299-4, J5 SSQ-120-01-L-D, J6 215299-4, Q1 2N7002, Q2 2N7002, Q3 Q_Photo_NPN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

Commit message: more autorouting
ugh please work i beg you
Parts:
- moved R1 18.1 mm to (77.0, 29.0), turned to 0 degrees
- moved USB1 1.00 mm to (68.0, 27.5)
Changed lines of the file:
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@@
   )
   (module ESP32bot:USB_C_Receptacle_HRO_TYPE-C-31-M-12 (layer F.Cu)
-    (at 69 27.5 180)
+    (at 68 27.5 180)
     (descr "USB Type-C receptacle for USB 2.0 and PD, http://www.krhro.com/uploads/soft/180320/1-1P320120243.pdf")
     (tags "usb usb-c 2.0 pd")
@@
   )
   (module Resistor_SMD:R_0603_1608Metric (layer F.Cu)
-    (at 59 31 180)
+    (at 77 29)
     (descr "Resistor SMD 0603 (1608 Metric), square (rectangular) end terminal, IPC_7351 nominal, (Body size source: IPC-SM-782 page 72, https://www.pcb-3d.com/wordpress/wp-content/uploads/ipc-sm-782a_amendment_1_and_2.pdf), generated with kicad-footprint-generator")
     (tags resistor)
@@
     (fp_line (start 1.48 -0.73) (end 1.48 0.73) (layer F.CrtYd) (width 0.05))
     (fp_line (start 1.48 0.73) (end -1.48 0.73) (layer F.CrtYd) (width 0.05))
-    (fp_text user %R (at 0 0 270) (layer F.Fab)
-      (effects (font (size 0.4 0.4) (thickness 0.06)))
-    )
-    (pad 2 smd roundrect (at 0.825 0 180) (size 0.8 0.95) (layers F.Cu F.Paste F.Mask) (roundrect_rratio 0.25)
-      (net 2 GND))
-    (pad 1 smd roundrect (at -0.825 0 180) (size 0.8 0.95) (layers F.Cu F.Paste F.Mask) (roundrect_rratio 0.25)
+    (fp_text user %R (at 0 0) (layer F.Fab)
+      (effects (font (size 0.4 0.4) (thickness 0.06)))
+    )
+    (pad 2 smd roundrect (at 0.825 0) (size 0.8 0.95) (layers F.Cu F.Paste F.Mask) (roundrect_rratio 0.25)
+      (net 2 GND))
+    (pad 1 smd roundrect (at -0.825 0) (size 0.8 0.95) (layers F.Cu F.Paste F.Mask) (roundrect_rratio 0.25)
       (net 57 "Net-(R1-Pad1)"))
     (model ${KISYS3DMOD}/Resistor_SMD.3dshapes/R_0603_1608Metric.wrl
