File: esp32pcbbot.sch (KiCad schematic (older format))
At the start: 44 parts, among them IC1 BMI055, J1 TB002-500-02BE, J2 TB002-500-02BE, J3 TB002-500-02BE, J4 215299-4, J5 SSQ-120-01-L-D, J6 215299-4, Q1 2N7002, Q2 2N7002, Q3 Q_Photo_NPN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

Commit message: cp2102 fixes
wow i screwed up
who would have thought
Parts:
- VR1: symbol LM3940IMP-3.3_NOPB:LM3940IMP-3.3_NOPB -> esp32pcbbot-rescue:LM3940IMP-3.3_NOPB-LM3940IMP-3.3_NOPB
Connections:
- net +3V3: no longer U2.7 (REGIN)
- net GND: no longer C4.2, C6.2, C8.2
- net VBUS: now also U2.7 (REGIN), U2.8 (VBUS)
Changed lines of the file:
@@
 (He Lives Within WIFI)
 $Comp
-L LM3940IMP-3.3_NOPB:LM3940IMP-3.3_NOPB VR1
+L esp32pcbbot-rescue:LM3940IMP-3.3_NOPB-LM3940IMP-3.3_NOPB VR1
 U 1 1 62706A8B
 P 2700 1250
@@
 	3600 2450 3600 2550
 Wire Wire Line
-	3600 2550 4000 2550
-Wire Wire Line
-	4100 2550 4100 2650
-Wire Wire Line
-	4000 2650 4000 2550
-Connection ~ 4000 2550
-Wire Wire Line
-	4000 2550 4100 2550
-Wire Wire Line
-	2350 3000 2350 3400
+	2350 3000 2350 3250
 Wire Wire Line
 	7000 1650 7000 1450
@@
 	1    0    0    -1
 $EndComp
-Connection ~ 11200 10550
-Wire Wire Line
-	11200 10550 11200 10800
 $Comp
 L SamacSys_Parts:EEEFC1V331P C7
@@
 	1    0    0    -1
 $EndComp
-Wire Wire Line
-	11200 10150 11200 10550
 $Comp
 L SamacSys_Parts:EEEFC1V331P C6
@@
 	1    0    0    -1
 $EndComp
-Connection ~ 10350 10550
-Wire Wire Line
-	10350 10550 10350 10800
 $Comp
 L SamacSys_Parts:EEEFC1V331P C5
@@
 	1    0    0    -1
 $EndComp
-Wire Wire Line
-	10350 10150 10350 10550
 $Comp
 L SamacSys_Parts:EEEFC1V331P C4
@@
 	1    0    0    -1
 $EndComp
-Connection ~ 9450 10550
-Wire Wire Line
-	9450 10550 9450 10800
 $Comp
 L SamacSys_Parts:EEEFC1V331P C3
@@
 $EndComp
 Wire Wire Line
-	9450 10150 9450 10550
-Wire Wire Line
 	9850 10550 9650 10550
 Wire Wire Line
@@
 Wire Wire Line
 	13950 3900 13950 4050
+Wire Wire Line
+	3600 3250 2800 3250
+Connection ~ 2350 3250
+Wire Wire Line
+	2350 3250 2350 3400
+Wire Wire Line
+	11200 10150 11200 10800
+Wire Wire Line
+	10350 10150 10350 10800
+Wire Wire Line
+	9450 10150 9450 10800
+Wire Wire Line
+	4100 2550 4100 2650
+Wire Wire Line
+	3600 2550 4100 2550
+Wire Wire Line
+	4000 2650 2800 2650
+Wire Wire Line
+	2800 2650 2800 3250
+Connection ~ 2800 3250
+Wire Wire Line
+	2800 3250 2350 3250
 $EndSCHEMATC

Commit message: more chaos
Parts:
- VR1: symbol esp32pcbbot-rescue:LM3940IMP-3.3_NOPB-LM3940IMP-3.3_NOPB -> LM3940IMP-3.3_NOPB:LM3940IMP-3.3_NOPB
Connections:
- net +3V3: now also U2.7 (REGIN)
- net GND: now also C4.2, C6.2, C8.2
- net VBUS: no longer U2.7 (REGIN)
Changed lines of the file:
@@
 (He Lives Within WIFI)
 $Comp
-L esp32pcbbot-rescue:LM3940IMP-3.3_NOPB-LM3940IMP-3.3_NOPB VR1
+L LM3940IMP-3.3_NOPB:LM3940IMP-3.3_NOPB VR1
 U 1 1 62706A8B
 P 2700 1250
@@
 	5900 1450 5900 3350
 Wire Wire Line
-	1750 3300 2000 3300
-Wire Wire Line
-	2000 3300 2000 4500
-Wire Wire Line
-	1750 4500 1850 4500
-Wire Wire Line
-	1750 4400 1850 4400
-Wire Wire Line
-	1850 4400 1850 4500
-Connection ~ 1850 4500
-Wire Wire Line
-	1850 4500 2000 4500
-Wire Wire Line
-	2350 3400 1750 3400
-Wire Wire Line
-	2350 3400 2350 4300
-Wire Wire Line
 	2350 4300 2300 4300
 Wire Wire Line
@@
 	2900 3350 3600 3350
 Wire Wire Line
-	1750 4000 1900 4000
-Wire Wire Line
-	1900 4000 1900 3800
-Connection ~ 1900 3800
-Wire Wire Line
-	1900 3800 2900 3800
-Wire Wire Line
 	2700 3700 2700 3450
 Wire Wire Line
 	2700 3450 3600 3450
 Wire Wire Line
-	1750 3900 2200 3900
-Wire Wire Line
-	2200 3900 2200 3700
-Connection ~ 2200 3700
-Wire Wire Line
-	2200 3700 2700 3700
-Wire Wire Line
 	2500 3600 2500 4550
 Wire Wire Line
 	2950 4200 2950 4550
 Wire Wire Line
-	2000 4500 2000 4950
-Connection ~ 2000 4500
-Wire Wire Line
 	2500 4850 2500 4950
 Wire Wire Line
 	2500 4950 2450 4950
-Connection ~ 2000 4950
 Wire Wire Line
 	2000 4950 2000 5300
@@
 Wire Wire Line
 	3600 2450 3600 2550
+Wire Wire Line
+	3600 2550 4000 2550
+Wire Wire Line
+	4100 2550 4100 2650
+Wire Wire Line
+	4000 2650 4000 2550
+Connection ~ 4000 2550
+Wire Wire Line
+	4000 2550 4100 2550
 Wire Wire Line
 	2350 3000 2350 3250
@@
 Wire Wire Line
 	15450 6850 15650 6850
-Connection ~ 2350 3400
 Connection ~ 7000 1650
 Wire Wire Line
@@
 	1    0    0    -1
 $EndComp
+Connection ~ 11200 10550
+Wire Wire Line
+	11200 10550 11200 10800
 $Comp
 L SamacSys_Parts:EEEFC1V331P C7
@@
 	1    0    0    -1
 $EndComp
+Wire Wire Line
+	11200 10150 11200 10550
 $Comp
 L SamacSys_Parts:EEEFC1V331P C6
@@
 	1    0    0    -1
 $EndComp
+Connection ~ 10350 10550
+Wire Wire Line
+	10350 10550 10350 10800
 $Comp
 L SamacSys_Parts:EEEFC1V331P C5
@@
 	1    0    0    -1
 $EndComp
+Wire Wire Line
+	10350 10150 10350 10550
 $Comp
 L SamacSys_Parts:EEEFC1V331P C4
@@
 	1    0    0    -1
 $EndComp
+Connection ~ 9450 10550
+Wire Wire Line
+	9450 10550 9450 10800
 $Comp
 L SamacSys_Parts:EEEFC1V331P C3
@@
 $EndComp
 Wire Wire Line
+	9450 10150 9450 10550
+Wire Wire Line
 	9850 10550 9650 10550
 Wire Wire Line
@@
 Wire Wire Line
 	2300 5750 2200 5750
-Connection ~ 2300 4300
-Wire Wire Line
-	2300 4300 1750 4300
 Wire Wire Line
 	750  3600 750  5950
@@
 	650  6050 800  6050
 Wire Wire Line
-	650  3800 1900 3800
-Wire Wire Line
 	600  3700 600  6150
 Wire Wire Line
 	600  6150 800  6150
-Wire Wire Line
-	600  3700 2200 3700
 Wire Wire Line
 	650  6050 650  6750
@@
 	7000 1900 9600 1900
 $Comp
-L power:GNDPWR #PWR?
+L power:GNDPWR #PWR0147
 U 1 1 628DA39C
 P 14400 4050
-F 0 "#PWR?" H 14400 3850 50  0001 C CNN
+F 0 "#PWR0147" H 14400 3850 50  0001 C CNN
 F 1 "GNDPWR" H 14404 3896 50  0000 C CNN
 F 2 "" H 14400 4000 50  0001 C CNN
@@
 	13950 3900 13950 4050
 Wire Wire Line
-	3600 3250 2800 3250
+	3600 3250 2350 3250
 Connection ~ 2350 3250
 Wire Wire Line
-	2350 3250 2350 3400
-Wire Wire Line
-	11200 10150 11200 10800
-Wire Wire Line
-	10350 10150 10350 10800
-Wire Wire Line
-	9450 10150 9450 10800
-Wire Wire Line
-	4100 2550 4100 2650
-Wire Wire Line
-	3600 2550 4100 2550
-Wire Wire Line
-	4000 2650 2800 2650
-Wire Wire Line
-	2800 2650 2800 3250
-Connection ~ 2800 3250
-Wire Wire Line
-	2800 3250 2350 3250
+	650  3800 2900 3800
+Wire Wire Line
+	600  3700 2700 3700
+Wire Wire Line
+	2350 3250 2350 4300
 $EndSCHEMATC

Commit message: update TODO
added things to do
Connections:
- net +3V3: now also U2.9 (~RSTb)
- net +5V: no longer U2.9 (~RSTb)
Changed lines of the file:
@@
-$EndComp
-$Comp
-L power:+5V #PWR0102
-U 1 1 625E73F9
-P 3250 2950
-F 0 "#PWR0102" H 3250 2800 50  0001 C CNN
-F 1 "+5V" H 3265 3123 50  0000 C CNN
-F 2 "" H 3250 2950 50  0001 C CNN
-F 3 "" H 3250 2950 50  0001 C CNN
-	1    3250 2950
-	1    0    0    -1
 $EndComp
 $Comp
@@
 	2700 3450 3600 3450
 Wire Wire Line
-	2500 3600 2500 4550
+	2500 4500 2500 4550
 Wire Wire Line
 	2950 4200 2950 4550
@@
 	3600 3050 3250 3050
 Wire Wire Line
-	3250 3050 3250 2950
-Wire Wire Line
 	4100 5250 4100 5900
 Wire Wire Line
@@
 	3600 2450 3600 2550
 Wire Wire Line
-	3600 2550 4000 2550
-Wire Wire Line
 	4100 2550 4100 2650
-Wire Wire Line
-	4000 2650 4000 2550
-Connection ~ 4000 2550
-Wire Wire Line
-	4000 2550 4100 2550
 Wire Wire Line
 	2350 3000 2350 3250
@@
 	2300 5750 2200 5750
 Wire Wire Line
-	750  3600 750  5950
+	750  4500 750  5950
 Wire Wire Line
 	750  5950 800  5950
 Wire Wire Line
-	750  3600 2500 3600
-Wire Wire Line
-	1400 4200 1400 5200
-Wire Wire Line
-	1400 5200 2650 5200
+	750  4500 2500 4500
+Wire Wire Line
+	3300 4200 3300 5200
+Wire Wire Line
+	3300 5200 2650 5200
 Wire Wire Line
 	2650 5200 2650 6250
@@
 	2650 6250 2200 6250
 Wire Wire Line
-	1400 4200 2950 4200
+	3300 4200 2950 4200
 Wire Wire Line
 	650  3800 650  6050
@@
 Wire Wire Line
 	13950 3900 13950 4050
-Wire Wire Line
-	3600 3250 2350 3250
 Connection ~ 2350 3250
 Wire Wire Line
@@
 Wire Wire Line
 	2350 3250 2350 4300
+Wire Wire Line
+	3600 2550 4000 2550
+Wire Wire Line
+	3250 2550 3600 2550
+Wire Wire Line
+	3250 2550 3250 3050
+Connection ~ 3600 2550
+Wire Wire Line
+	2350 3250 3600 3250
+Wire Wire Line
+	4000 2650 4000 2550
+Connection ~ 4000 2550
+Wire Wire Line
+	4000 2550 4100 2550
 $EndSCHEMATC
