File: esp32pcbbot.kicad_sch (KiCad schematic)
At the start: 41 parts, among them IC1 BMI055, J1 TB002-500-02BE, J2 TB002-500-02BE, J3 TB002-500-02BE, J4 215299-4, J5 SSQ-120-01-L-D, J6 215299-4, Q1 2N7002, Q2 2N7002, U1 ESP32-WROOM-32E-Espressif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

Commit message: i did the LED
glow
Parts:
- added D? (x2): LED, symbol Device:LED
- added R? (x2): R, symbol Device:R
Connections:
- net GND: now also D?.1 (K), D?.1 (K)
- net at U2.18 (~{RXT}/GPIO.1): now also R?.1
- net at U2.19 (~{TXT}/GPIO.0): now also R?.1
- new net: D?.2 (A), R?.2 (x2)
