File: esp32pcbbot.kicad_sch (KiCad schematic)
At the start: 39 parts, among them IC1 BMI055, J1 TB002-500-02BE, J2 TB002-500-02BE, J3 TB002-500-02BE, J4 215299-4, J5 SSQ-120-01-L-D, J6 215299-4, Q1 2N7002, Q2 2N7002, U1 ESP32-WROOM-32E-Espressif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

Commit message: cp2102 circuitry layout
made it more ✨pretty✨
Connections:
- net GND: no longer R1.2, R2.2, USB1.A1 (GND), USB1.A12 (GND), USB1.B1 (GND), USB1.B12 (GND), USB1.S1 (SHIELD), USB1.S2 (SHIELD), USB1.S3 (SHIELD), USB1.S4 (SHIELD)
- net at Q1.2 (S), U2.28 (~{DTR}): now also R4.2; no longer R4.1
- net at Q2.1 (G): now also R4.1; no longer R4.2
- net at R2.1: now also R1.2, USB1.A1 (GND), USB1.A12 (GND), USB1.B1 (GND), USB1.B12 (GND), USB1.S1 (SHIELD), USB1.S2 (SHIELD), USB1.S3 (SHIELD), USB1.S4 (SHIELD); no longer USB1.B5 (CC2)
- new net: R2.2, USB1.B5 (CC2)
- no-connect marks 0 -> 1
Other:
- note added: "To GPIO header"
- moved on the sheet: Q1, Q2, R2, R3, R4, USB1, VR1

Commit message: H bridge and resistors?? idk???
i dont know wtf i did but it helped
oh hey i did stuff on the LED indecators
wait i think i also fixed the power circuitry for the H bridge motor driver
Parts:
- added D1, D2: LED, symbol Device:LED
- added R7, R8: 47, symbol Device:R
Connections:
- net +5V: now also U3.16 (VCC1)
- net GND: now also R1.2, R2.1, USB1.A1 (GND), USB1.A12 (GND), USB1.B1 (GND), USB1.B12 (GND), USB1.S1 (SHIELD), USB1.S2 (SHIELD), USB1.S3 (SHIELD), USB1.S4 (SHIELD), D1.1 (K), D2.1 (K)
- net at U2.18 (~{RXT}/GPIO.1): now also R7.1
- net at U2.19 (~{TXT}/GPIO.0): now also R8.1
- net at S2.2: now also S2.5, U3.8 (VCC2); no longer U3.16 (VCC1)
- new net: D2.2 (A), R8.2
- new net: D1.2 (A), R7.2
Other:
- note added: "USB circuitry"
- note added: "USB-C port"
- note added: "Yellow LEDs"
